Commit message: working on beaker bot states

File: gym/beaker.urdf (robot description, URDF)
Before this commit: robot myfirst, 3 links, 2 joints
Links:
- added link axle_link; visual cylinder length=0.17 radius=.01
- added link face_link; visual box size=0.05 0.01 0.05
- link base_link: mass 1.765 -> 1.767
- link left_wheel: mass 0.1 -> 0.09
- link right_wheel: mass 0.1 -> 0.09
Joints:
- added joint axle_joint: type fixed, parent base_link, child axle_link, axis 1 0 0
- added joint face_joint: type fixed, parent base_link, child face_link

Commit message: figured out how to calculate theta dot in pybullet

File: gym/beaker.urdf (robot description, URDF)
Before this commit: robot myfirst, 5 links, 4 joints
Links:
- removed link base_link
- removed link face_link
- added link body, mass 1.767; collision box size=0.1016 0.0254 0.6604; visual box size=0.1016 0.0254 0.6604
- added link face; visual box size=0.05 0.01 0.05
Joints:
- joint axle_joint: parent base_link -> body
- joint base_to_left_wheel: parent base_link -> body
- joint base_to_right_wheel: parent base_link -> body
- joint face_joint: child face_link -> face; parent base_link -> body

Commit message: making the robot easier to see

File: gym/beaker.urdf (robot description, URDF)
Before this commit: robot beaker, 5 links, 4 joints
Links:
- removed link axle_link
- added link left_wheel_stripe; visual box size=0.01 0.01 0.08
- added link right_wheel_stripe; visual box size=0.01 0.01 0.08
- link body: geometry collision box size=0.1016 0.0254 0.6604; visual box size=0.1016 0.0254 0.6604
Joints:
- removed joint axle_joint
- added joint left_wheel_to_stripe: type fixed, parent left_wheel, child left_wheel_stripe
- added joint right_wheel_to_stripe: type fixed, parent right_wheel, child right_wheel_stripe
- joint base_to_left_wheel: origin xyz=0.09398 0.0 0.01905 -> xyz=-0.09398 0.0 0.01905
- joint base_to_right_wheel: origin xyz=-0.09398 0.0 0.01905 -> xyz=0.09398 0.0 0.01905

Commit message: still messing around

File: gym/beaker.urdf (robot description, URDF)
Before this commit: robot beaker, 6 links, 5 joints
Links:
- link face: mass None -> 0
- link left_wheel_stripe: mass None -> 0
- link right_wheel_stripe: mass None -> 0

Commit message: removed old controllers

File: gym/beaker.urdf (robot description, URDF)
Before this commit: robot beaker, 6 links, 5 joints
Links:
- link body: mass 1.767 -> 0.001767
- link left_wheel: mass 0.09 -> 0.0009
- link right_wheel: mass 0.09 -> 0.0009

Commit message: fix small inconsistency in beaker.urdf

File: gym/beaker.urdf (robot description, URDF)
Before this commit: robot beaker, 6 links, 5 joints
Links:
- link body: mass 0.001767 -> 1.767
- link left_wheel: mass 0.0009 -> 0.09
- link right_wheel: mass 0.0009 -> 0.09

Commit message: finishes to the beaker URDF builder

File: gym/beaker.urdf (robot description, URDF)
Before this commit: robot beaker, 6 links, 5 joints
Links:
- removed link left_wheel
- removed link left_wheel_stripe
- removed link right_wheel
- removed link right_wheel_stripe
- added link leftWheel, mass .1; collision cylinder length=0.0254 radius=0.042; visual cylinder length=0.0254 radius=0.042
- added link leftWheelIndicator, mass .0000; visual box size=0.01 0.01 0.01
- added link rightWheel, mass .1; collision cylinder length=0.0254 radius=0.042; visual cylinder length=0.0254 radius=0.042
- added link rightWheelIndicator, mass .0000; visual box size=0.01 0.01 0.01
Joints:
- removed joint left_wheel_to_stripe
- removed joint right_wheel_to_stripe
- added joint indicatorToleftWheel: type fixed, parent leftWheel, child leftWheelIndicator, origin xyz=0 0.042 0
- added joint indicatorTorightWheel: type fixed, parent rightWheel, child rightWheelIndicator, origin xyz=0 0.042 0
- joint base_to_left_wheel: child left_wheel -> leftWheel; limit (none) -> lower=-0.0756 upper=0.0756 effort=1000 velocity=1000; origin xyz=-0.09398 0.0 0.01905 -> xyz=-0.09398 0 0.01905; type continuous -> revolute
- joint base_to_right_wheel: child right_wheel -> rightWheel; limit (none) -> lower=-0.0756 upper=0.0756 effort=1000 velocity=1000; origin xyz=0.09398 0.0 0.01905 -> xyz=0.09398 0 0.01905; type continuous -> revolute

Commit message: fix urdf builder

File: gym/beaker.urdf (robot description, URDF)
Before this commit: robot beaker, 6 links, 5 joints
Links:
- removed link leftWheel
- removed link rightWheel
- added link left_wheel, mass .1; collision cylinder length=0.0254 radius=0.042; visual cylinder length=0.0254 radius=0.042
- added link right_wheel, mass .1; collision cylinder length=0.0254 radius=0.042; visual cylinder length=0.0254 radius=0.042
Joints:
- removed joint indicatorToleftWheel
- removed joint indicatorTorightWheel
- added joint indicator_to_left_wheel: type fixed, parent left_wheel, child leftWheelIndicator, origin xyz=0 0.042 0
- added joint indicator_to_right_wheel: type fixed, parent right_wheel, child rightWheelIndicator, origin xyz=0 0.042 0
- joint base_to_left_wheel: child leftWheel -> left_wheel
- joint base_to_right_wheel: child rightWheel -> right_wheel

Commit message: working on urdf again

File: gym/beaker.urdf (robot description, URDF)
Before this commit: robot beaker, 6 links, 5 joints
Links:
- removed link face
- removed link leftWheelIndicator
- removed link rightWheelIndicator
- added link left_gear, mass .00001; visual cylinder length=0.02 radius=0.03
- added link right_gear, mass .00001; visual cylinder length=0.02 radius=0.03
Joints:
- removed joint base_to_left_wheel
- removed joint base_to_right_wheel
- removed joint face_joint
- removed joint indicator_to_left_wheel
- removed joint indicator_to_right_wheel
- added joint base_to_left_gear: type continuous, parent body, child left_gear, origin xyz=-0.061 0 0.01905, axis 1 0 0
- added joint base_to_right_gear: type continuous, parent body, child right_gear, origin xyz=0.061 0 0.01905, axis 1 0 0
- added joint gear_to_left_wheel: type revolute, parent left_gear, child left_wheel, origin xyz=-0.09398 0 0.01905, axis 1 0 0, limit lower=-0.0756 upper=0.0756 effort=1000 velocity=1000
- added joint gear_to_right_wheel: type revolute, parent right_gear, child right_wheel, origin xyz=0.09398 0 0.01905, axis 1 0 0, limit lower=-0.0756 upper=0.0756 effort=1000 velocity=1000

Commit message: closer to solving this horrible mystery

File: gym/beaker.urdf (robot description, URDF)
Before this commit: robot beaker, 5 links, 4 joints
Links:
- link body: geometry collision box size=0.1016 0.0254 0.6604; visual box size=0.1016 0.0254 0.6604
- link left_gear: mass .00001 -> 0.1; geometry collision cylinder length=0.01 radius=0.04; visual cylinder length=0.01 radius=0.04
- link left_wheel: mass .1 -> 0.1
- link right_gear: mass .00001 -> 0.1; geometry collision cylinder length=0.01 radius=0.04; visual cylinder length=0.01 radius=0.04
- link right_wheel: mass .1 -> 0.1
Joints:
- removed joint base_to_left_gear
- removed joint base_to_right_gear
- added joint body_to_left_gear: type continuous, parent body, child left_gear, origin xyz=-0.061 0 0.01905, axis 1 0 0
- added joint body_to_right_gear: type continuous, parent body, child right_gear, origin xyz=0.061 0 0.01905, axis 1 0 0

Commit message: use the non backlash urdf file

File: gym/beaker.urdf (robot description, URDF)
Before this commit: robot beaker, 5 links, 4 joints
Links:
- removed link left_gear
- removed link right_gear
Joints:
- removed joint base_to_left_gear
- removed joint base_to_right_gear
- removed joint gear_to_left_wheel
- removed joint gear_to_right_wheel
- added joint base_to_left_wheel: type revolute, parent body, child left_wheel, origin xyz=-0.09398 0 0.01905, axis 1 0 0, limit lower=-0.0756 upper=0.0756 effort=1000 velocity=1000
- added joint base_to_right_wheel: type revolute, parent body, child right_wheel, origin xyz=0.09398 0 0.01905, axis 1 0 0, limit lower=-0.0756 upper=0.0756 effort=1000 velocity=1000
